File: KiCad/TS_Core.kicad_sch (KiCad schematic)
At the start: 42 parts, among them J1 USB Serial, J2 M5StickC Hat, J3 AQM1248A, J4 TinyStick_Ext1, J5 TinyStick_Ext2, J6 Grove Connector, J7 LCD BackLight, Q2 AO3400A, SW1 Tactile, SW1 Tactile(Side)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

Commit message: update 5 buttons
Parts:
- removed J4: TinyStick_Ext1, Connector_PinSocket_2.54mm:PinSocket_1x08_P2.54mm_Vertical, symbol Connector:Conn_01x08_Socket
- added J4: TinyStick_Ext1, Connector_PinSocket_2.54mm:PinSocket_1x07_P2.54mm_Vertical, symbol Connector:Conn_01x07_Socket
- added SW1: Tactile, JSB01_Lib:SW-SMD_4P-L4.5-W4.5-P3.00-LS7.5, symbol JSB01_Lib:SW_Tactile4P
- J5: footprint Connector_PinSocket_2.54mm:PinSocket_1x07_P2.54mm_Vertical -> Connector_PinSocket_2.54mm:PinSocket_1x06_P2.54mm_Vertical; symbol Connector:Conn_01x07_Socket -> Connector:Conn_01x06_Socket
- renumbered SW5 to SW6, SW6 to SW7
Connections:
- net +3V3: now also J4.1 (Pin_1)
- net +5V: now also J4.7 (Pin_7); no longer J5.7 (Pin_7)
- net GND: now also SW1.3, SW1.4
- net PA4: now also J4.2 (Pin_2)
- net PA5: now also J4.3 (Pin_3)
- net PA6: now also J4.4 (Pin_4)
- net PB6: now also U2.12 (INT1)
- net RXD: now also J4.5 (Pin_5)
- net SW4: now also SW1.1, SW1.2; no longer SW1.1
- net TXD: now also J4.6 (Pin_6)
- net PB7 renamed SW5
- net SW5: now also SW1.1
- no-connect marks 5 -> 4
Other:
- moved on the sheet: SW1
